File: scripts/corner_case/corner_case.kicad_pcb (KiCad board)
At the start: 2 copper layers, 80 x 104 mm, 46 parts, among them J1 TYPE-C-31-M-12, Q1 2SA812, Q2 2SA812, Q3 2SA812, Q4 2SA812, Q5 2SA812, Q6 2SA812, Q7 HT7133S (SOT-23 -CW numbering), U1 LM358DR2G, U10 NE555P, U2 LM358DR2G, U3 LM358DR2G, U4 RFX2401C, U5 LMV321IDBVR, U6 MT3608, U7 LMV321IDBVR wrong pick, U8 AMS1117-3.3, U9 L78M05ABDT-TR

Commit message: test(jlcfootprint): in-stock stand-ins for D8 and D10; bidirectional D13; gate compares axis parts modulo 180
JLC no longer stocks C1978115 (D8) and C1981006 (D10), so the board could
not be placed. D10 is now C707468 SMF7.0A, the same SMF -RD footprint with
pin 1 = C; D8 is C1973411 SMF51A-E3-08, an SMF -R-FD part whose symbol pins
are just 1/2, so the name token alone decides (C1978115's data had drifted
to the same case as D9 anyway). D13 C2857328 SMF15CA adds the -BI case with
the A1/A2 pin functions KiCad's D_TVS symbol gives it; the resolver settles
a bidirectional token before looking for a KiCad reference pad, because
A1/A2 read as two anodes. The gate compares axis-aligned parts modulo 180:
a non-polar part 180 degrees from JLC's angle is the same placement.
Board regenerated (47 parts); report rows D8, D10 changed and D13 added.

Co-Authored-By: Claude Fable 5.1 <noreply@anthropic.com>
Parts:
- added D13: SMF15CA (-BI bidirectional; D_TVS pins A1/A2), Diode_SMD:D_SMF, F.Cu at (58.0, 94.0)
- D10: value VTVS12ASMF-M-18 -> SMF7.0A (RD; pin 1 = C)
- D8: value VTVS17ASMF-M3-08 -> SMF51A-E3-08 (-R-FD; numeric symbol pins)
