File: tests/fixtures/jlcfootprint/boards/pin_functions_and_marks/pin_functions_and_marks.kicad_pcb (KiCad board)
At the start: 2 copper layers, 80 x 44 mm, 16 parts, among them U1 3095K (JLC numbers the tab 3;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, U2 3095K (functions IN/D/S as on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, U3 3095K placed at 90, U4 MC78M08CDTRKG (TL-CW; tab is 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, U5 3095K without pin functions: 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

Commit message: docs(jlcfootprint): say what the resolver and its gate do, and document them in the README
The comments and docstrings of polarity, fit, resolver and resolving, the
four gate tools (validate_board, check_live_adapter,
make_corner_case_board, truth_from_presses) and the resolver's and the
gate's tests now explain the code on their own: no design-note section
numbers, milestone names, bead ids, dates, review notes or narration of
earlier states.  Calibration stays as measurements over EasyEDA's library
or on the committed gate boards: the FD/RD token's agreement with the "+"
marks on electrolytic cans and molded-chip tantalums, and SHAPE_MARGIN
against the gate boards' two-pad parts and the recorded coin-cell holder.

jlcfootprint/README.md gains "Judging a part" (the three alignment paths,
the polarity vote and its tie rule, the second pairing, the fit grades and
statuses, the body caveat and the package origin) and "The gate" (the two
boards, what the truth files mean, how validate_board reproduces JLC's
placement preview and how to run it), in place of the resolver's line
under "What comes next".  Its module table lists the four modules.

The gate data's prose says what the boards show, without dates, milestone
names or the names of other boards: the notes in the three truth CSVs,
truth_presses.csv's header, and the value text of three parts in the
second board's cases.csv and its board file (no code reads a Value field
or a note).  The board's C8 value still named the part C1969735 replaced
and said its token and marks disagree; it now names TMCP1A106MTRF, as
cases.csv does, and says they agree, as the resolver finds.

Two prose strings in code change with them: validate_board's --flip-y
help cited a design-note section, and the gate test's skip reason (never
reached: the truth file is committed) cited a plan task.

One code change, not in behaviour: Optional annotations follow upstream's
convention (its CLAUDE.md: "Use Optional[X] instead of X | None"), 53 of
the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
Parts:
- C5: value TAJB105K035RNJ (-R-RD: the token is wrong; the + marks decide) -> TAJB105K035RNJ (-R-RD: the token and the + marks agree)
- C8: value TPCR106K016R1800 (-FD: token and + marks disagree; preview decides) -> TMCP1A106MTRF (-FD: the token and both + marks say 0; preview 0)
- U2: value 3095K (functions IN/D/S as on test-Placements U12; G by elimination) -> 3095K (functions IN/D/S; G by elimination)
Changed lines of the file:
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@@
 			)
 		)
-		(property "Value" "TPCR106K016R1800 (-FD: token and + marks disagree; preview decides)"
+		(property "Value" "TMCP1A106MTRF (-FD: the token and both + marks say 0; preview 0)"
 			(at 0 1.58 0)
 			(layer "F.Fab")
@@
 			)
 		)
-		(property "Value" "3095K (functions IN/D/S as on test-Placements U12; G by elimination)"
+		(property "Value" "3095K (functions IN/D/S; G by elimination)"
 			(at 0 4.5 0)
 			(layer "F.Fab")
@@
 			)
 		)
-		(property "Value" "TAJB105K035RNJ (-R-RD: the token is wrong; the + marks decide)"
+		(property "Value" "TAJB105K035RNJ (-R-RD: the token and the + marks agree)"
 			(at 0 2.35 0)
 			(layer "F.Fab")
